File: esp8266.sch (KiCad schematic (older format))
At the start: 15 parts, among them P1 VIN, P2 CONN_01X08, P3 CONN_01X08, P4 CONN_01X06, SW1 SW_PUSH, SW2 SW_PUSH, U1 APE8865N-33-HF-3

Commit message: spread PCB
Connections:
- net GPIO0: now also P3.5 (P5); no longer P3.3 (P3)
- net GPIO4: now also P3.4 (P4); no longer P3.5 (P5)
- net GPIO5: now also P3.3 (P3); no longer P3.4 (P4)
Changed lines of the file:
@@
 LIBS:valves
 LIBS:esp8266
+LIBS:esp8266-cache
 EELAYER 25 0
 EELAYER END
@@
 RXD
 Text Label 3900 5050 2    60   ~ 0
+GPIO5
+Text Label 3900 5150 2    60   ~ 0
+GPIO4
+Text Label 3900 5250 2    60   ~ 0
 GPIO0
-Text Label 3900 5150 2    60   ~ 0
-GPIO5
-Text Label 3900 5250 2    60   ~ 0
-GPIO4
 Text Label 3900 5350 2    60   ~ 0
 GPIO2
